Commit message: add antenna to robot

File: src/ur5e_dual_horn_description/urdf/dual_horn.urdf.xacro (robot description, xacro)
@@ -1,44 +1,38 @@
 <?xml version="1.0"?>
 <robot xmlns:xacro="http://www.ros.org/wiki/xacro" name="ur5e_dual_horn">
-	<xacro:arg name="parent_link" default="tool0" />
-	<xacro:arg name="prefix" default="" />
-	<xacro:arg name="mesh_file" default="package://ur5e_dual_horn_description/meshes/dual_horn.stl" />
-	<xacro:arg name="mount_xyz" default="0 0 0" />
-	<xacro:arg name="mount_rpy" default="0 0 0" />
-    % Antenna mount links
-    <link name="$(arg parent_link)" />
-    % Joint with respect to plan
-    <link name="$(arg prefix)central_antenna_link" />
-	<link name="$(arg prefix)dual_horn_link">
-		<visual>
-			<origin xyz="0 0 0" rpy="0 0 0" />
-			<geometry>
-				<mesh filename="$(arg mesh_file)" scale="0.001 0.001 0.001" />
-			</geometry>
-			<material name="dark_gray">
-				<color rgba="0.2 0.2 0.2 1.0" />
-			</material>
-		</visual>
-		<collision>
-			<origin xyz="0 0 0" rpy="0 0 0" />
-			<geometry>
-				<mesh filename="$(arg mesh_file)" scale="0.001 0.001 0.001" />
-			</geometry>
-		</collision>
-		<inertial>
-			<origin xyz="0 0 0" rpy="0 0 0" />
-			<mass value="0.2" />
-			<inertia ixx="0.0001" ixy="0.0" ixz="0.0" iyy="0.0001" iyz="0.0" izz="0.0001" />
-		</inertial>
-	</link>
-	<joint name="$(arg prefix)dual_horn_fixed_joint" type="fixed">
-		<parent link="$(arg parent_link)" />
-		<child link="$(arg prefix)dual_horn_link" />
-		<origin xyz="$(arg mount_xyz)" rpy="$(arg mount_rpy)" />
-	</joint>
-    <joint name="$(arg prefix)central_antenna_joint" type="fixed">
-		<parent link="$(arg prefix)dual_horn_link" />
-		<child link="$(arg prefix)central_antenna_link" />
-		<origin xyz="0.0 0.0 -0.16" rpy="0.0 0.0 0.0" />
-	</joint>
+  <xacro:macro name="dual_horn" params="parent_link prefix mesh_file mount_xyz mount_rpy">
+    <link name="${prefix}antenna_center_link"/>
+    <link name="${prefix}dual_horn_link">
+      <visual>
+        <origin xyz="0 0 0" rpy="0 0 0" />
+        <geometry>
+          <mesh filename="${mesh_file}" scale="0.001 0.001 0.001" />
+        </geometry>
+        <material name="dark_gray">
+          <color rgba="0.2 0.2 0.2 1.0" />
+        </material>
+      </visual>
+      <collision>
+        <origin xyz="0 0 0" rpy="0 0 0" />
+        <geometry>
+          <mesh filename="${mesh_file}" scale="0.001 0.001 0.001" />
+        </geometry>
+      </collision>
+      <inertial>
+        <origin xyz="0 0 0" rpy="0 0 0" />
+        <mass value="0.2" />
+        <inertia ixx="0.0001" ixy="0.0" ixz="0.0" iyy="0.0001" iyz="0.0" izz="0.0001" />
+      </inertial>
+    </link>
+    <joint name="${prefix}dual_horn_fixed_joint" type="fixed">
+      <parent link="${parent_link}" />
+      <child link="${prefix}dual_horn_link" />
+      <origin xyz="${mount_xyz}" rpy="${mount_rpy}" />
+    </joint>
+    <joint name="${prefix}antenna_center_joint" type="fixed">
+      <parent link="${prefix}dual_horn_link" />
+      <child link="${prefix}antenna_center_link" />
+      <origin xyz="0.0 0.0 -0.16" rpy="${mount_rpy}" />
+    </joint>
+  </xacro:macro>
 </robot>
