Commit message: connection to simulator

File: src/ur5e_dual_horn_description/urdf/ur5e_dual_horn.xacro (robot description, xacro)
@@ -14,6 +14,31 @@
 	<xacro:arg name="mount_rpy" default="0.0 -3.14159 1.5708" />
 	<xacro:arg name="mesh_file" default="package://ur5e_dual_horn_description/meshes/dual_horn.stl" />
+	<xacro:arg name="transmission_hw_interface" default="" />
+	<xacro:arg name="headless_mode" default="false" />
+	<xacro:arg name="robot_ip" default="0.0.0.0" />
+	<xacro:arg name="script_filename" default="$(find ur5e_dual_horn_description)/ur_programs/connect_sim_robot.script" />
+	<xacro:arg name="output_recipe_filename" default="$(find ur5e_dual_horn_description)/ur_programs/connect_sim_robot.old0" />
+	<xacro:arg name="input_recipe_filename" default="$(find ur5e_dual_horn_description)/ur_programs/connect_sim_robot.old1" />
+	<xacro:arg name="reverse_ip" default="0.0.0.0" />
+	<xacro:arg name="script_command_port" default="50004" />
+	<xacro:arg name="reverse_port" default="50001" />
+	<xacro:arg name="script_sender_port" default="50002" />
+	<xacro:arg name="trajectory_port" default="50003" />
+	<xacro:arg name="use_tool_communication" default="false" />
+	<xacro:arg name="tool_voltage" default="0" />
+	<xacro:arg name="tool_parity" default="0" />
+	<xacro:arg name="tool_baud_rate" default="115200" />
+	<xacro:arg name="tool_stop_bits" default="1" />
+	<xacro:arg name="tool_rx_idle_chars" default="1.5" />
+	<xacro:arg name="tool_tx_idle_chars" default="3.5" />
+	<xacro:arg name="tool_device_name" default="/tmp/ttyUR" />
+	<xacro:arg name="tool_tcp_port" default="54321" />
+	<xacro:arg name="use_mock_hardware" default="false" />
+	<xacro:arg name="mock_sensor_commands" default="false" />
+	<xacro:arg name="initial_positions_file" default="$(find ur5e_dual_horn_description)/config/initial_positions.yaml" />
+	<xacro:arg name="use_ros2_control" default="true" />
 	<xacro:include filename="$(find ur_description)/urdf/ur_macro.xacro" />
 	<xacro:include filename="$(find ur5e_dual_horn_description)/urdf/dual_horn.urdf.xacro" />
+	<xacro:include filename="$(find ur5e_dual_horn_description)/urdf/ur5e_dual_horn_ros2_control.xacro" />
 	<link name="world" />
 	<xacro:ur_robot
@@ -33,3 +58,34 @@
 		mount_xyz="$(arg mount_xyz)"
 		mount_rpy="$(arg mount_rpy)" />
+	<xacro:if value="$(arg use_ros2_control)">
+		<xacro:ur5e_dual_horn_ros2_control
+			name="FakeSystem"
+			tf_prefix="$(arg tf_prefix)"
+			kinematics_params="$(arg kinematics_params)"
+			transmission_hw_interface="$(arg transmission_hw_interface)"
+			use_fake_hardware="$(arg use_fake_hardware)"
+			com_port="$(arg com_port)"
+			use_tool_communication="$(arg use_tool_communication)"
+			tool_voltage="$(arg tool_voltage)"
+			tool_parity="$(arg tool_parity)"
+			tool_baud_rate="$(arg tool_baud_rate)"
+			tool_stop_bits="$(arg tool_stop_bits)"
+			tool_rx_idle_chars="$(arg tool_rx_idle_chars)"
+			tool_tx_idle_chars="$(arg tool_tx_idle_chars)"
+			tool_device_name="$(arg tool_device_name)"
+			tool_tcp_port="$(arg tool_tcp_port)"
+			robot_ip="$(arg robot_ip)"
+			script_filename="$(arg script_filename)"
+			output_recipe_filename="$(arg output_recipe_filename)"
+			input_recipe_filename="$(arg input_recipe_filename)"
+			reverse_ip="$(arg reverse_ip)"
+			script_command_port="$(arg script_command_port)"
+			reverse_port="$(arg reverse_port)"
+			script_sender_port="$(arg script_sender_port)"
+			trajectory_port="$(arg trajectory_port)"
+			headless_mode="$(arg headless_mode)"
+			use_mock_hardware="$(arg use_mock_hardware)"
+			mock_sensor_commands="$(arg mock_sensor_commands)"
+			initial_positions_file="$(arg initial_positions_file)" />
+	</xacro:if>
 </robot>

File: src/ur5e_dual_horn_moveit_config/config/ur5e_dual_horn.urdf.xacro (robot description, xacro)
@@ -1,9 +1,43 @@
 <?xml version="1.0"?>
 <robot xmlns:xacro="http://www.ros.org/wiki/xacro" name="ur5e_dual_horn">
-    <xacro:arg name="initial_positions_file" default="initial_positions.yaml" />
-    <!-- Import ur5e_dual_horn urdf file -->
-    <xacro:include filename="$(find ur5e_dual_horn_description)/urdf/ur5e_dual_horn.xacro" />
-    <!-- Import control_xacro -->
-    <xacro:include filename="ur5e_dual_horn.ros2_control.xacro" />
-    <xacro:ur5e_dual_horn_ros2_control name="FakeSystem" initial_positions_file="$(arg initial_positions_file)"/>
+    <xacro:arg name="name" default="ur" />
+    <xacro:arg name="ur_type" default="ur5e" />
+    <xacro:arg name="tf_prefix" default="" />
+    <xacro:arg name="joint_limit_params" default="$(find ur_description)/config/$(arg ur_type)/joint_limits.yaml" />
+    <xacro:arg name="kinematics_params" default="$(find ur_description)/config/$(arg ur_type)/default_kinematics.yaml" />
+    <xacro:arg name="physical_params" default="$(find ur_description)/config/$(arg ur_type)/physical_parameters.yaml" />
+    <xacro:arg name="visual_params" default="$(find ur_description)/config/$(arg ur_type)/visual_parameters.yaml" />
+    <xacro:arg name="use_fake_hardware" default="true" />
+    <xacro:arg name="com_port" default="/dev/ttyUSB0" />
+    <xacro:arg name="parent" default="world" />
+    <xacro:arg name="mount_xyz" default="0.0 0.0 0.037" />
+    <xacro:arg name="mount_rpy" default="0.0 -3.14159 1.5708" />
+    <xacro:arg name="mesh_file" default="package://ur5e_dual_horn_description/meshes/dual_horn.stl" />
+    <xacro:arg name="initial_positions_file" default="$(find ur5e_dual_horn_description)/config/initial_positions.yaml" />
+    <xacro:arg name="use_ros2_control" default="true" />
+    <xacro:include filename="$(find ur_description)/urdf/ur_macro.xacro" />
+    <xacro:include filename="$(find ur5e_dual_horn_description)/urdf/dual_horn.urdf.xacro" />
+    <xacro:include filename="$(find ur5e_dual_horn_description)/urdf/ur5e_dual_horn_ros2_control.xacro" />
+    <link name="world" />
+    <xacro:ur_robot
+        name="$(arg name)"
+        tf_prefix="$(arg tf_prefix)"
+        parent="$(arg parent)"
+        joint_limits_parameters_file="$(arg joint_limit_params)"
+        kinematics_parameters_file="$(arg kinematics_params)"
+        physical_parameters_file="$(arg physical_params)"
+        visual_parameters_file="$(arg visual_params)">
+        <origin xyz="0 0 0" rpy="0 0 0" />
+    </xacro:ur_robot>
+    <xacro:dual_horn
+        parent_link="$(arg tf_prefix)tool0"
+        prefix="$(arg tf_prefix)"
+        mesh_file="$(arg mesh_file)"
+        mount_xyz="$(arg mount_xyz)"
+        mount_rpy="$(arg mount_rpy)" />
+    <xacro:if value="$(arg use_ros2_control)">
+        <xacro:ur5e_dual_horn_ros2_control
+            name="FakeSystem"
+            initial_positions_file="$(arg initial_positions_file)" />
+    </xacro:if>
 </robot>
